File: amp_nanopi.brd (EAGLE design)
At the start: 87.1 x 64 mm, 11 parts, among them J1 MF-CON-2.54mm-01x02, J2 MF-CON-2.54mm-01x02, J3 MF-CON-2.54mm-01x02, X1 B3P-VH-2, X2 B3P-VH-2

Commit message: przygotowanie do wyslania do pcbs.io
Parts:
- flipped X3 to the top
- flipped X4 to the top
Connections:
- net GND: now also X3.12, X3.15, X4.1; no longer X3.14, X3.9, X4.12
- net N$1: now also X4.6; no longer X4.7
