File: amp_nanopi.sch (EAGLE design)
At the start: 11 parts, among them J1 MF-CON-2.54mm-01x02, J2 MF-CON-2.54mm-01x02, J3 MF-CON-2.54mm-01x02, X2 B3P-VH-2, X3 B3P-VH-2

Commit message: dostosowanie do nowego projektu safe_pi_shutdown
Parts:
- removed SV1: (no value), con-lstb:MA12-2
- added X1: B3P-VH-2, jst-vh:B3P-VH-2
- X3: value B3P-VH-2 -> (none); device jst-vh:B3P-VH-2 -> con-lstb:MA12-2
- renumbered SV2 to X4, U$1 to U1
Connections:
- net GND: now also X3.14, X3.20, X3.6, X3.9; no longer SV1.14, SV1.20, SV1.6, SV1.9
- net N$4: now also X1.1; no longer X3.1
- net N$6: now also X1.2; no longer X3.2
Changed lines of the file:
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@@
 <parts>
 <part name="S1" library="switch-omron" deviceset="31-XX" device=""/>
-<part name="U$1" library="meanwell_irm_v5" deviceset="IRM_05/10" device=""/>
+<part name="U1" library="meanwell_irm_v5" deviceset="IRM_05/10" device=""/>
 <part name="F1" library="fuse" deviceset="FUSE" device="SH22,5"/>
 <part name="F2" library="fuse" deviceset="FUSE" device="SH22,5"/>
 <part name="X2" library="jst-vh" deviceset="B3P-VH-2" device=""/>
-<part name="X3" library="jst-vh" deviceset="B3P-VH-2" device=""/>
-<part name="SV1" library="con-lstb" deviceset="MA12-2" device=""/>
-<part name="SV2" library="con-lstb" deviceset="MA12-1" device=""/>
+<part name="X1" library="jst-vh" deviceset="B3P-VH-2" device=""/>
+<part name="X3" library="con-lstb" deviceset="MA12-2" device=""/>
+<part name="X4" library="con-lstb" deviceset="MA12-1" device=""/>
 <part name="J1" library="MF_Connectors" deviceset="CON_01X02" device="_PTH_2.54MM" value="MF-CON-2.54mm-01x02"/>
 <part name="J2" library="MF_Connectors" deviceset="CON_01X02" device="_PTH_2.54MM" value="MF-CON-2.54mm-01x02"/>
@@
 <instances>
 <instance part="S1" gate="1" x="50.8" y="78.74" rot="MR0"/>
-<instance part="U$1" gate="G$1" x="86.36" y="43.18" rot="R180"/>
+<instance part="U1" gate="G$1" x="86.36" y="43.18" rot="R180"/>
 <instance part="F1" gate="G$1" x="109.22" y="50.8"/>
 <instance part="F2" gate="G$1" x="124.46" y="60.96" rot="R90"/>
 <instance part="X2" gate="G$1" x="139.7" y="71.12"/>
-<instance part="X3" gate="G$1" x="139.7" y="45.72"/>
-<instance part="SV1" gate="1" x="30.48" y="38.1" rot="R180"/>
-<instance part="SV2" gate="1" x="-7.62" y="35.56" rot="MR180"/>
+<instance part="X1" gate="G$1" x="139.7" y="45.72"/>
+<instance part="X3" gate="1" x="30.48" y="38.1" rot="R180"/>
+<instance part="X4" gate="1" x="-7.62" y="35.56" rot="MR180"/>
 <instance part="J1" gate="G$1" x="20.32" y="83.82" rot="R180"/>
 <instance part="J2" gate="G$1" x="60.96" y="30.48" rot="R270"/>
@@
 <net name="VCC" class="0">
 <segment>
-<pinref part="U$1" gate="G$1" pin="V+"/>
+<pinref part="U1" gate="G$1" pin="V+"/>
 <label x="68.58" y="35.56" size="1.778" layer="95"/>
 <pinref part="J2" gate="G$1" pin="PIN1"/>
@@
 <wire x1="22.86" y1="83.82" x2="48.26" y2="83.82" width="0.1524" layer="91"/>
 <wire x1="48.26" y1="83.82" x2="48.26" y2="71.12" width="0.1524" layer="91"/>
-<pinref part="U$1" gate="G$1" pin="V-"/>
+<pinref part="U1" gate="G$1" pin="V-"/>
 <wire x1="73.66" y1="50.8" x2="50.8" y2="50.8" width="0.1524" layer="91"/>
-<pinref part="SV1" gate="1" pin="6"/>
+<pinref part="X3" gate="1" pin="6"/>
 <wire x1="38.1" y1="45.72" x2="50.8" y2="45.72" width="0.1524" layer="91"/>
 <wire x1="50.8" y1="45.72" x2="50.8" y2="50.8" width="0.1524" layer="91"/>
-<pinref part="SV1" gate="1" pin="14"/>
+<pinref part="X3" gate="1" pin="14"/>
 <wire x1="38.1" y1="35.56" x2="50.8" y2="35.56" width="0.1524" layer="91"/>
 <wire x1="50.8" y1="35.56" x2="50.8" y2="45.72" width="0.1524" layer="91"/>
-<pinref part="SV1" gate="1" pin="20"/>
+<pinref part="X3" gate="1" pin="20"/>
 <wire x1="38.1" y1="27.94" x2="50.8" y2="27.94" width="0.1524" layer="91"/>
 <wire x1="50.8" y1="27.94" x2="50.8" y2="35.56" width="0.1524" layer="91"/>
-<pinref part="SV1" gate="1" pin="9"/>
+<pinref part="X3" gate="1" pin="9"/>
 <wire x1="22.86" y1="40.64" x2="20.32" y2="40.64" width="0.1524" layer="91"/>
 <wire x1="20.32" y1="40.64" x2="20.32" y2="20.32" width="0.1524" layer="91"/>
@@
 <junction x="50.8" y="35.56"/>
 <junction x="50.8" y="45.72"/>
-<pinref part="SV2" gate="1" pin="12"/>
+<pinref part="X4" gate="1" pin="12"/>
 <wire x1="0" y1="20.32" x2="20.32" y2="20.32" width="0.1524" layer="91"/>
 <junction x="20.32" y="20.32"/>
@@
 <junction x="124.46" y="50.8"/>
 <wire x1="124.46" y1="50.8" x2="124.46" y2="45.72" width="0.1524" layer="91"/>
-<pinref part="X3" gate="G$1" pin="1"/>
+<pinref part="X1" gate="G$1" pin="1"/>
 <wire x1="124.46" y1="45.72" x2="139.7" y2="45.72" width="0.1524" layer="91"/>
 </segment>
@@
 <segment>
 <pinref part="F1" gate="G$1" pin="1"/>
-<pinref part="U$1" gate="G$1" pin="AC/L"/>
+<pinref part="U1" gate="G$1" pin="AC/L"/>
 <wire x1="104.14" y1="50.8" x2="99.06" y2="50.8" width="0.1524" layer="91"/>
 </segment>
@@
 <wire x1="139.7" y1="43.18" x2="124.46" y2="43.18" width="0.1524" layer="91"/>
 <wire x1="124.46" y1="43.18" x2="124.46" y2="35.56" width="0.1524" layer="91"/>
-<pinref part="U$1" gate="G$1" pin="AC/N"/>
+<pinref part="U1" gate="G$1" pin="AC/N"/>
 <wire x1="124.46" y1="35.56" x2="99.06" y2="35.56" width="0.1524" layer="91"/>
 <wire x1="124.46" y1="35.56" x2="147.32" y2="35.56" width="0.1524" layer="91"/>
@@
 <junction x="124.46" y="35.56"/>
 <pinref part="X2" gate="G$1" pin="2"/>
-<pinref part="X3" gate="G$1" pin="2"/>
+<pinref part="X1" gate="G$1" pin="2"/>
 </segment>
 </net>
@@
 <net name="N$1" class="0">
 <segment>
-<pinref part="SV2" gate="1" pin="7"/>
+<pinref part="X4" gate="1" pin="7"/>
 <wire x1="0" y1="33.02" x2="15.24" y2="33.02" width="0.1524" layer="91"/>
 <wire x1="15.24" y1="33.02" x2="15.24" y2="66.04" width="0.1524" layer="91"/>

Commit message: przygotowanie do wyslania do pcbs.io
Connections:
- net GND: now also X3.12, X3.15, X4.1; no longer X3.14, X3.9, X4.12
- net N$1: now also X4.6; no longer X4.7
Other:
- moved on the sheet: X3, X4
Changed lines of the file:
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@@
 </class>
 <class number="1" name="230V" width="2.032" drill="1.27">
-<clearance class="1" value="5.08"/>
+<clearance class="1" value="2.54"/>
 </class>
 </classes>
@@
 <instance part="X2" gate="G$1" x="139.7" y="71.12"/>
 <instance part="X1" gate="G$1" x="139.7" y="45.72"/>
-<instance part="X3" gate="1" x="30.48" y="38.1" rot="R180"/>
-<instance part="X4" gate="1" x="-7.62" y="35.56" rot="MR180"/>
+<instance part="X3" gate="1" x="30.48" y="35.56" rot="MR0"/>
+<instance part="X4" gate="1" x="-7.62" y="33.02"/>
 <instance part="J1" gate="G$1" x="20.32" y="83.82" rot="R180"/>
 <instance part="J2" gate="G$1" x="60.96" y="30.48" rot="R270"/>
@@
 <pinref part="U1" gate="G$1" pin="V-"/>
 <wire x1="73.66" y1="50.8" x2="50.8" y2="50.8" width="0.1524" layer="91"/>
-<pinref part="X3" gate="1" pin="6"/>
 <wire x1="38.1" y1="45.72" x2="50.8" y2="45.72" width="0.1524" layer="91"/>
 <wire x1="50.8" y1="45.72" x2="50.8" y2="50.8" width="0.1524" layer="91"/>
-<pinref part="X3" gate="1" pin="14"/>
 <wire x1="38.1" y1="35.56" x2="50.8" y2="35.56" width="0.1524" layer="91"/>
 <wire x1="50.8" y1="35.56" x2="50.8" y2="45.72" width="0.1524" layer="91"/>
-<pinref part="X3" gate="1" pin="20"/>
 <wire x1="38.1" y1="27.94" x2="50.8" y2="27.94" width="0.1524" layer="91"/>
 <wire x1="50.8" y1="27.94" x2="50.8" y2="35.56" width="0.1524" layer="91"/>
-<pinref part="X3" gate="1" pin="9"/>
-<wire x1="22.86" y1="40.64" x2="20.32" y2="40.64" width="0.1524" layer="91"/>
 <wire x1="20.32" y1="40.64" x2="20.32" y2="20.32" width="0.1524" layer="91"/>
 <wire x1="20.32" y1="20.32" x2="20.32" y2="15.24" width="0.1524" layer="91"/>
@@
 <junction x="50.8" y="35.56"/>
 <junction x="50.8" y="45.72"/>
-<pinref part="X4" gate="1" pin="12"/>
-<wire x1="0" y1="20.32" x2="20.32" y2="20.32" width="0.1524" layer="91"/>
-<junction x="20.32" y="20.32"/>
 <pinref part="S1" gate="1" pin="P"/>
 <wire x1="50.8" y1="73.66" x2="50.8" y2="71.12" width="0.1524" layer="91"/>
@@
 <wire x1="12.7" y1="68.58" x2="50.8" y2="68.58" width="0.1524" layer="91"/>
 <junction x="50.8" y="68.58"/>
+<pinref part="X4" gate="1" pin="1"/>
+<wire x1="0" y1="20.32" x2="20.32" y2="20.32" width="0.1524" layer="91"/>
+<junction x="20.32" y="20.32"/>
+<pinref part="X3" gate="1" pin="15"/>
+<wire x1="20.32" y1="40.64" x2="22.86" y2="40.64" width="0.1524" layer="91"/>
+<pinref part="X3" gate="1" pin="6"/>
+<pinref part="X3" gate="1" pin="12"/>
+<pinref part="X3" gate="1" pin="20"/>
 </segment>
 </net>
@@
 <net name="N$1" class="0">
 <segment>
-<pinref part="X4" gate="1" pin="7"/>
-<wire x1="0" y1="33.02" x2="15.24" y2="33.02" width="0.1524" layer="91"/>
 <wire x1="15.24" y1="33.02" x2="15.24" y2="66.04" width="0.1524" layer="91"/>
 <pinref part="J3" gate="G$1" pin="PIN1"/>
 <wire x1="15.24" y1="66.04" x2="12.7" y2="66.04" width="0.1524" layer="91"/>
+<pinref part="X4" gate="1" pin="6"/>
+<wire x1="0" y1="33.02" x2="15.24" y2="33.02" width="0.1524" layer="91"/>
 </segment>
 </net>
